File: termo.sch (KiCad schematic (older format))
At the start: 17 parts, among them J1 USB_A, J2 Conn_01x04_Female, J3 Conn_02x05_Odd_Even, U1 AMS1117, U3 HDC1080, Y1 Crystal

Commit message: Final layout
Parts:
- removed J3: Conn_02x05_Odd_Even, Connector_PinHeader_1.00mm:PinHeader_2x05_P2.67mm_Vertical, symbol Connector_Generic:Conn_02x05_Odd_Even
- added J3: ISP, Connector_PinHeader_2.54mm:PinHeader_2x03_P2.54mm_Vertical, symbol Connector_Generic:Conn_02x03_Odd_Even
- added J4: PA, Connector_PinHeader_2.54mm:PinHeader_1x08_P2.54mm_Vertical, symbol Connector:Conn_01x08_Female
- added J5: PB, Connector_PinHeader_2.54mm:PinHeader_1x08_P2.54mm_Vertical, symbol Connector:Conn_01x08_Female
- added J6: PC, Connector_PinHeader_2.54mm:PinHeader_1x08_P2.54mm_Vertical, symbol Connector:Conn_01x08_Female
- added J7: PD, Connector_PinHeader_2.54mm:PinHeader_1x08_P2.54mm_Vertical, symbol Connector:Conn_01x08_Female
- added J8: PWR, Connector_PinHeader_2.54mm:PinHeader_1x06_P2.54mm_Vertical, symbol Connector:Conn_01x06_Female
- added J9: PA, Connector_PinHeader_2.54mm:PinHeader_1x02_P2.54mm_Vertical, symbol Connector:Conn_01x02_Female
- added R5: R, Resistor_SMD:R_0805_2012Metric, symbol Device:R
- renumbered C_block to C_block1, U_mega to U_mega1
Connections:
- net labels added: aref, avcc
- wire segments 78 -> 129
- no-connect marks 1 -> 0
Other:
- moved on the sheet: C3, C4
